File: vr_module.kicad_pcb (KiCad board)
At the start: 4 copper layers, 20.3 x 22.9 mm, 44 parts, among them J1 Conn_01x07, U1 MAX9142, U2 NC7SB3157P6X, U3 74HC02, U4 NC7SB3157P6X, U5 SRV05-4, U6 MCP6004

Commit message: KiCAD version sync no real changes yet. Just opens in KiCAD with out version complaints.
Other:
- net class Default removed
